File: esp12-breakout.kicad_pcb (KiCad board)
At the start: 2 copper layers, 50 x 50 mm, 32 parts, among them CON1 USB-MINI-B, P1 CONN_14, SW1 SW_PUSH, U1 CH340G, U2 ESP-12, U3 LM1117-3.3, X1 CRYSTAL

Commit message: Workshop 3 Warmup
Parts:
- added D5: DIODE, w_smd_diode:sod123, F.Cu at (186.7, 134.6)
- added P2: CONN_4, connect:SIL-4, F.Cu at (175.3, 133.3)
- added P3: CONN_4, connect:SIL-4, F.Cu at (182.2, 142.2)
- added P4: CONN_4, connect:SIL-4, F.Cu at (174.6, 137.8)
- C5, C8: value CP1 -> 10u
- C6, C7: value C -> 100n
- R2: value R -> 10k
- moved SW1 51.1 mm to (92.1, 48.3)
- moved U1 47.1 mm to (187.3, 39.4)
- moved C8 27.5 mm to (168.3, 44.5)
- moved C5 24.5 mm to (120.7, 44.5)
- moved RP4 13.9 mm to (128.9, 54.0)
- moved R1 12.1 mm to (153.7, 49.5)
- moved R2 11.2 mm to (153.7, 52.1)
- moved RP3 10.9 mm to (134.6, 47.6)
- moved R6 10.9 mm to (153.7, 54.6)
- moved C7 9.36 mm to (150.5, 49.5)
- moved RP2 8.49 mm to (134.6, 57.1)
- moved RP1 8.44 mm to (134.6, 52.7)
- moved R3 8.19 mm to (150.5, 52.1)
- moved R7 7.71 mm to (150.5, 54.6)
- moved C6 6.98 mm to (147.3, 49.5)
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Routing:
- net +5V: track 3.81 -> 7.58 mm
- net Net-(CON1-Pad1): track 5.25 -> 4.61 mm

Commit message: Workshop 3
Parts:
- added 1PIN: P***, connect:1pin, F.Cu at (139.1, 81.3)
- added 1PIN: P***, connect:1pin, F.Cu at (139.1, 125.1)
- added 1PIN: P***, connect:1pin, F.Cu at (182.9, 125.1)
- moved C1 109.3 mm to (158.1, 110.5), turned to 270 degrees
- moved SW1 104.2 mm to (164.5, 123.2), turned to 180 degrees
- moved P1 90.7 mm to (183.5, 97.2), turned to 270 degrees
- moved C3 85.3 mm to (158.1, 114.3), turned to 270 degrees
- moved U1 80.1 mm to (153.0, 111.8), turned to 90 degrees
- moved C5 77.8 mm to (141.6, 119.4)
- moved RP5 75.3 mm to (179.1, 113.0), turned to 180 degrees
- moved RP4 71.4 mm to (179.1, 104.8), turned to 180 degrees
- moved C4 70.1 mm to (160.7, 117.5), turned to 90 degrees
- moved C6 66.2 mm to (142.2, 115.6), turned to 180 degrees
- moved RP3 64.7 mm to (179.1, 94.6), turned to 180 degrees
- moved C8 63.1 mm to (141.6, 101.6)
- moved C2 56.7 mm to (158.1, 105.4), turned to 90 degrees
- moved C7 56.5 mm to (142.2, 105.4), turned to 180 degrees
- moved R1 55.2 mm to (153.7, 104.8), turned to 270 degrees
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Connections:
- RP4 pad 1: Net-(RP4-Pad1) -> GPIO5
- RP4 pad 2: Net-(RP4-Pad2) -> GPIO4
- RP4 pad 3: Net-(RP4-Pad3) -> SLCK
- RP4 pad 4: Net-(RP4-Pad4) -> MOSI
- U2 pad 13: Net-(RP4-Pad1) -> MOSI
- U2 pad 14: Net-(RP4-Pad2) -> SLCK
- U2 pad 19: Net-(RP4-Pad3) -> GPIO4
- U2 pad 20: Net-(RP4-Pad4) -> GPIO5
Routing:
- net +3.3V: track 0.00 -> 153.6 mm, vias 0 -> 7
- net Reset: track 0.00 -> 73.1 mm, vias 0 -> 3
- net RXD: track 0.00 -> 71.2 mm, vias 0 -> 3
- net TXD: track 0.00 -> 68.3 mm, vias 0 -> 3
- net +5V: track 7.58 -> 71.8 mm, vias 0 -> 3
- net Net-(RP2-Pad4): track 0.00 -> 40.5 mm
- net Net-(RP2-Pad3): track 0.00 -> 39.5 mm
- net Net-(RP2-Pad2): track 0.00 -> 38.1 mm
- net Net-(RP2-Pad1): track 0.00 -> 33.6 mm
- net Net-(RP3-Pad1): track 0.00 -> 29.8 mm, vias 0 -> 2
- net GPIO15: track 0.00 -> 29.6 mm
- net GPIO2: track 0.00 -> 29.4 mm
- net Net-(RP3-Pad2): track 0.00 -> 28.1 mm, vias 0 -> 2
- net GPIO5: track 0.00 -> 26.9 mm
- net GPIO4: track 0.00 -> 26.1 mm
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- added copper zone on F.Cu, net GND
Other:
- net class Default: via_dia 0.6 -> 0.4; via_drill 0.4 -> 0.25
