File: esp12-breakout.sch (KiCad schematic (older format))
At the start: 27 parts

Commit message: Second session
Parts:
- removed P?: CONN_12, symbol CONN_12
- removed R?: R, symbol R
- removed RP? (x2): R_PACK8, symbol R_PACK8
- removed U?: CH340H/T, symbol CH340H/T
- added D1, D2, D4: LED, led:LED-0603, symbol LED
- added P1: CONN_14, connect:SIL-14, symbol CONN_14
- added RP1, RP2, RP3, RP4, RP5: R_PACK4, smd_resistors:r_cat16-4, symbol R_PACK4
- added U?: CH340G, SOP-16, symbol CH340G
- C1, C2: renamed from C?; value C -> 22p; footprint (none) -> libcms:SM0603
- C3: renamed from C?; value C -> 100n; footprint (none) -> libcms:SM0603
- C4, C6, C7: renamed from C?; footprint (none) -> libcms:SM0603
- C5, C8: renamed from C?; footprint (none) -> smd_capacitors:c_elec_5x5.3
- CON1: renamed from CON?; footprint (none) -> connect:USB_MINI_B
- D3: renamed from D?; footprint (none) -> led:LED-0603
- L1: renamed from L?; footprint (none) -> libcms:SM0805
- R1, R2, R3, R4, R5, R6, R7: renamed from R?; footprint (none) -> libcms:SM0603
- SW1: renamed from SW?; footprint (none) -> discret:SW_PUSH_SMALL
- X1: renamed from X?; footprint (none) -> discret:HC-49V
- gave numbers to parts that had none: 2
Connections:
- net +3.3V: now also RP1.2 (P2), RP1.3 (P3), RP1.4 (P4), U?.16 (VCC), U?.4 (V3)
- net +5V: now also RP1.1 (P1)
- net GND: now also D4.2 (K), U?.1 (GND)
- net RXD: now also D2.2 (K), U?.3 (RX)
- net TXD: now also D1.2 (K), U?.2 (TX)
- net UD+: now also U?.5 (D+)
- net UD-: now also U?.6 (D-)
- net at U2.10 (MISO): now also RP3.2 (P2)
- net at U2.11 (GPIO9): now also RP3.3 (P3)
- net at U2.12 (GPIO10): now also RP3.4 (P4)
- net at U2.13 (MOSI): now also RP4.1 (P1)
- net at U2.14 (SLCK): now also RP4.2 (P2)
- net GPIO15: now reaches R7.1, U2.16 (GPIO15)
- net GPIO15: now also RP5.2 (P2)
- net GPIO2: now reaches R6.1, U2.17 (GPIO2)
- net GPIO2: now also RP5.1 (P1)
- net at U2.19 (GPIO4): now also RP4.3 (P3)
- net at U2.2 (ADC): now also RP2.1 (P1)
- net at U2.20 (GPIO5): now also RP4.4 (P4)
- net at U2.5 (GPIO14): now also RP2.2 (P2)
- net at U2.6 (GPIO12): now also RP2.3 (P3)
- net at U2.7 (GPIO17): now also RP2.4 (P4)
- net at U2.9 (CS0): now also RP3.1 (P1)
- net at D3.1 (A): now also RP1.7 (R2)
- net at C2.1, X1.2: now also U?.8 (XO)
- net at R2.2: now also U?.13 (DTR)
- net at R1.2: now also U?.14 (RTS)
- net at C1.1, X1.1: now also U?.7 (XI)
- new net: D1.1 (A), RP1.5 (R4)
- new net: D2.1 (A), RP1.6 (R3)
- new net: D4.1 (A), RP1.8 (R1)
- new net: P1.1 (P1), RP2.8 (R1)
- new net: P1.10 (P10), RP4.7 (R2)
- new net: P1.11 (P11), RP4.6 (R3)
- new net: P1.12 (P12), RP4.5 (R4)
- new net: P1.13 (P13), RP5.8 (R1)
- new net: P1.14 (P14), RP5.7 (R2)
- new net: P1.2 (P2), RP2.7 (R2)
- new net: P1.3 (P3), RP2.6 (R3)
- new net: P1.4 (P4), RP2.5 (R4)
- new net: P1.5 (P5), RP3.8 (R1)
- new net: P1.6 (P6), RP3.7 (R2)
- new net: P1.7 (P7), RP3.6 (R3)
- new net: P1.8 (P8), RP3.5 (R4)
- new net: P1.9 (P9), RP4.8 (R1)
Other:
- moved on the sheet: C1, C2, C3, C5, C6, C7, C8, D3, R1, R2, U3, X1

Commit message: Workshop 3 Warmup
Parts:
- added D5: DIODE, w_smd_diode:sod123, symbol DIODE
- added P2, P3, P4: CONN_4, connect:SIL-4, symbol CONN_4
- C5, C8: value CP1 -> 10u
- C6, C7: value C -> 100n
- R2: value R -> 10k
- U1: renamed from U?; footprint SOP-16 -> CH340G:SOP-16
- U2: footprint (none) -> esp12-f:ESP-12F
- U3: footprint TO-39 -> LM1117:sot223
Connections:
- net +3.3V: now also D5.1 (A), P3.1 (P1), P3.2 (P2), P3.3 (P3), P3.4 (P4)
- net +5V: now also D5.2 (K), P2.1 (P1), P2.2 (P2), P2.3 (P3), P2.4 (P4)
- net GND: now also P4.1 (P1), P4.2 (P2), P4.3 (P3), P4.4 (P4)
Other:
- moved on the sheet: C5, C6, C7, C8, U3

Commit message: Workshop 3
Connections:
- net GPIO5: now reaches RP4.1 (P1)
- net GPIO5: now also U2.20 (GPIO5); no longer U2.13 (MOSI)
- net GPIO4: now reaches RP4.2 (P2)
- net GPIO4: now also U2.19 (GPIO4); no longer U2.14 (SLCK)
- net SLCK: now reaches RP4.3 (P3)
- net SLCK: now also U2.14 (SLCK); no longer U2.19 (GPIO4)
- net MOSI: now reaches RP4.4 (P4)
- net MOSI: now also U2.13 (MOSI); no longer U2.20 (GPIO5)
Other:
- moved on the sheet: RP4, RP5
Changed lines of the file:
@@
 $EndComp
 Wire Wire Line
-	8450 1600 8700 1600
-Wire Wire Line
-	8700 1600 9150 1600
-Wire Wire Line
-	9150 1600 9200 1600
+	8450 1600 9200 1600
 Wire Wire Line
 	8700 1600 8700 1750
 Connection ~ 8700 1600
 Wire Wire Line
-	10000 1600 10100 1600
-Wire Wire Line
-	10100 1600 10600 1600
-Wire Wire Line
-	10600 1600 10850 1600
+	10000 1600 10850 1600
 Wire Wire Line
 	10600 1750 10600 1600
@@
 $EndComp
 Wire Wire Line
-	10100 1150 10100 1600
-Wire Wire Line
-	10100 1600 10100 1750
+	10100 1150 10100 1750
 Connection ~ 10100 1600
 Wire Wire Line
-	9150 1150 9150 1600
-Wire Wire Line
-	9150 1600 9150 1750
+	9150 1150 9150 1750
 Connection ~ 9150 1600
 Wire Wire Line
@@
 $EndComp
 Wire Wire Line
-	1000 1250 1000 1400
-Wire Wire Line
-	1000 1400 1000 1700
-Wire Wire Line
-	1000 1700 1000 1850
-Wire Wire Line
-	1000 1850 1000 2000
+	1000 1250 1000 2000
 Wire Wire Line
 	1000 1250 1150 1250
@@
 $EndComp
 Wire Wire Line
-	6050 5650 6100 5650
-Wire Wire Line
-	6100 5650 6250 5650
-Wire Wire Line
-	6050 5500 6100 5500
-Wire Wire Line
-	6100 5500 6250 5500
+	6050 5650 6250 5650
+Wire Wire Line
+	6050 5500 6250 5500
 Wire Wire Line
 	5550 5500 5450 5500
@@
 	6250 3150 6050 3150
 Wire Wire Line
-	5400 2950 5500 2950
-Wire Wire Line
-	5500 2950 6250 2950
+	5400 2950 6250 2950
 $Comp
 L R R4
@@
 	4650 3350 5550 3350
 Wire Wire Line
-	4650 2500 4650 2950
-Wire Wire Line
-	4650 2950 4650 3350
+	4650 2500 4650 3350
 $Comp
 L +3.3V #PWR016
@@
 Reset
 Wire Wire Line
-	5300 3150 5500 3150
-Wire Wire Line
-	5500 3150 5550 3150
+	5300 3150 5550 3150
 Wire Wire Line
 	5500 3150 5500 2950
@@
 $EndComp
 Wire Wire Line
-	5750 6650 5900 6650
-Wire Wire Line
-	5900 6650 6550 6650
+	5750 6650 6550 6650
 Wire Wire Line
 	5900 6650 5900 6800
@@
 	9050 4500 9050 3800
 Wire Wire Line
-	8250 4700 9250 4700
-Wire Wire Line
-	8250 4900 8450 4900
-Wire Wire Line
-	8450 4900 8450 4800
-Wire Wire Line
-	8450 4800 9250 4800
-Wire Wire Line
-	8250 5100 8550 5100
-Wire Wire Line
-	8550 5100 8550 4900
-Wire Wire Line
-	8550 4900 9250 4900
-Wire Wire Line
-	8250 5300 8650 5300
-Wire Wire Line
-	8650 5300 8650 5000
-Wire Wire Line
-	8650 5000 9250 5000
-Wire Wire Line
 	9650 3100 10300 3100
 Wire Wire Line
@@
 	9650 3400 10300 3400
 Wire Wire Line
-	9650 4700 9750 4700
+	9700 4700 9750 4700
 Wire Wire Line
 	9750 4700 9750 3900
@@
 	9750 3900 10300 3900
 Wire Wire Line
-	9650 4800 9850 4800
+	9700 4800 9850 4800
 Wire Wire Line
 	9850 4800 9850 4000
@@
 	9850 4000 10300 4000
 Wire Wire Line
-	9650 4900 9950 4900
+	9700 4900 9950 4900
 Wire Wire Line
 	9950 4900 9950 4100
@@
 	9950 4100 10300 4100
 Wire Wire Line
-	9650 5000 10050 5000
+	9700 5000 10050 5000
 Wire Wire Line
 	10050 5000 10050 4200
@@
 	1900 4600 2700 4600
 Wire Wire Line
-	1500 4850 1600 4850
-Wire Wire Line
-	1600 4850 1900 4850
+	1500 4850 1900 4850
 Wire Wire Line
 	1600 4850 1600 4800
@@
 	1600 4200 1600 4150
 Wire Wire Line
-	1500 4150 1600 4150
-Wire Wire Line
-	1600 4150 1900 4150
+	1500 4150 1900 4150
 $Comp
 L C C1
@@
 Connection ~ 1050 4850
 $Comp
-L GND #PWR020
+L GND #PWR019
 U 1 1 56D78E3E
 P 1050 5000
-F 0 "#PWR020" H 1050 5000 30  0001 C CNN
+F 0 "#PWR019" H 1050 5000 30  0001 C CNN
 F 1 "GND" H 1050 4930 30  0001 C CNN
 F 2 "" H 1050 5000 60  0000 C CNN
@@
 	2250 6050 2250 6250
 $Comp
-L +3.3V #PWR021
+L +3.3V #PWR020
 U 1 1 56E07094
 P 1850 5250
-F 0 "#PWR021" H 1850 5210 30  0001 C CNN
+F 0 "#PWR020" H 1850 5210 30  0001 C CNN
 F 1 "+3.3V" H 1862 5388 30  0000 C CNN
 F 2 "" H 1850 5250 60  0000 C CNN
@@
 	2250 6800 2250 6650
 $Comp
-L GND #PWR022
+L GND #PWR021
 U 1 1 56E07E07
 P 3100 6850
-F 0 "#PWR022" H 3100 6850 30  0001 C CNN
+F 0 "#PWR021" H 3100 6850 30  0001 C CNN
 F 1 "GND" H 3100 6780 30  0001 C CNN
 F 2 "" H 3100 6850 60  0000 C CNN
@@
 	2150 5250 2150 5500
 $Comp
-L +5V #PWR023
+L +5V #PWR022
 U 1 1 56E08263
 P 2150 5250
-F 0 "#PWR023" H 2150 5340 20  0001 C CNN
+F 0 "#PWR022" H 2150 5340 20  0001 C CNN
 F 1 "+5V" H 2143 5379 30  0000 C CNN
 F 2 "" H 2150 5250 60  0000 C CNN
@@
 	6100 5900 6100 5650
 Connection ~ 6100 5650
-Text GLabel 9100 5100 0    60   Input ~ 0
+Text GLabel 9150 5200 0    60   Input ~ 0
 GPIO2
-Text GLabel 9100 5250 0    60   Input ~ 0
+Text GLabel 9150 5350 0    60   Input ~ 0
 GPIO15
 Wire Wire Line
-	9100 5100 9250 5100
-Wire Wire Line
-	9100 5250 9150 5250
-Wire Wire Line
-	9150 5250 9150 5200
-Wire Wire Line
-	9150 5200 9250 5200
+	9150 5350 9250 5350
+Wire Wire Line
+	9250 5350 9250 5200
+Wire Wire Line
+	9250 5200 9300 5200
 $Comp
 L CONN_14 P1
@@
 $EndComp
 Wire Wire Line
-	9650 5100 10200 5100
+	9700 5100 10200 5100
 Wire Wire Line
 	10200 5100 10200 4300
@@
 	10200 4300 10300 4300
 Wire Wire Line
-	9650 5200 10300 5200
+	9700 5200 10300 5200
 Wire Wire Line
 	10300 5200 10300 4400
@@
 L R_PACK4 RP4
 U 1 1 56E0A065
-P 9450 5050
-F 0 "RP4" H 9450 5595 40  0000 C CNN
-F 1 "R_PACK4" H 9450 5517 40  0000 C CNN
-F 2 "smd_resistors:r_cat16-4" H 9450 5050 60  0001 C CNN
-F 3 "" H 9450 5050 60  0000 C CNN
-	1    9450 5050
+P 9500 5050
+F 0 "RP4" H 9500 5595 40  0000 C CNN
+F 1 "R_PACK4" H 9500 5517 40  0000 C CNN
+F 2 "smd_resistors:r_cat16-4" H 9500 5050 60  0001 C CNN
+F 3 "" H 9500 5050 60  0000 C CNN
+	1    9500 5050
 	1    0    0    -1
 $EndComp
@@
 L R_PACK4 RP5
 U 1 1 56E0A06B
-P 9450 5450
-F 0 "RP5" H 9450 5300 40  0000 C CNN
-F 1 "R_PACK4" H 9450 5400 40  0000 C CNN
-F 2 "smd_resistors:r_cat16-4" H 9450 5450 60  0001 C CNN
-F 3 "" H 9450 5450 60  0000 C CNN
-	1    9450 5450
+P 9500 5450
+F 0 "RP5" H 9500 5300 40  0000 C CNN
+F 1 "R_PACK4" H 9500 5400 40  0000 C CNN
+F 2 "smd_resistors:r_cat16-4" H 9500 5450 60  0001 C CNN
+F 3 "" H 9500 5450 60  0000 C CNN
+	1    9500 5450
 	1    0    0    -1
 $EndComp
@@
 $EndComp
 Wire Wire Line
-	1850 5250 1850 5450
-Wire Wire Line
-	1850 5450 1850 5500
-Wire Wire Line
-	1850 5450 1950 5450
-Wire Wire Line
-	1950 5450 2050 5450
+	1850 5250 1850 5500
+Wire Wire Line
+	1850 5450 2050 5450
 Wire Wire Line
 	1950 5450 1950 5500
@@
 	1650 3800 2700 3800
 Wire Wire Line
-	1050 3200 1050 4150
-Wire Wire Line
-	1050 4150 1050 4850
-Wire Wire Line
-	1050 4850 1050 5000
-Wire Wire Line
-	1050 3200 2500 3200
-Wire Wire Line
-	2500 3200 2700 3200
-$Comp
-L +3.3V #PWR024
+	1050 3200 1050 5000
+Wire Wire Line
+	1050 3200 2700 3200
+$Comp
+L +3.3V #PWR023
 U 1 1 56E0CBF4
 P 1650 3650
-F 0 "#PWR024" H 1650 3610 30  0001 C CNN
+F 0 "#PWR023" H 1650 3610 30  0001 C CNN
 F 1 "+3.3V" H 1662 3788 30  0000 C CNN
 F 2 "" H 1650 3650 60  0000 C CNN
@@
 Connection ~ 2500 3200
 Wire Wire Line
-	4000 2300 4000 2700
-Wire Wire Line
-	4000 2700 4000 3200
+	4000 2300 4000 3200
 Wire Wire Line
 	3500 2700 4000 2700
@@
 	4000 3200 3900 3200
 $Comp
-L +3.3V #PWR025
+L +3.3V #PWR024
 U 1 1 56E0D1F5
 P 4000 2300
-F 0 "#PWR025" H 4000 2260 30  0001 C CNN
+F 0 "#PWR024" H 4000 2260 30  0001 C CNN
 F 1 "+3.3V" H 4012 2438 30  0000 C CNN
 F 2 "" H 4000 2300 60  0000 C CNN
@@
 	4550 1450 4650 1450
 Wire Wire Line
-	4550 900  4550 1150
-Wire Wire Line
-	4550 1150 4550 1250
-Wire Wire Line
-	4550 1250 4550 1350
-Wire Wire Line
-	4550 1350 4550 1450
+	4550 900  4550 1450
 Wire Wire Line
 	4550 1150 4650 1150
@@
 	5650 1150 5550 1150
 Wire Wire Line
-	5550 900  5550 1150
-Wire Wire Line
-	5550 1150 5550 1250
-Wire Wire Line
-	5550 1250 5550 1350
-Wire Wire Line
-	5550 1350 5550 1450
+	5550 900  5550 1450
 Wire Wire Line
 	5550 1250 5650 1250
@@
 	6700 1150 6550 1150
 Wire Wire Line
-	6550 1150 6550 1250
-Wire Wire Line
-	6550 1250 6550 1350
-Wire Wire Line
-	6550 1350 6550 1450
-Wire Wire Line
-	6550 1450 6550 1600
+	6550 1150 6550 1600
 Wire Wire Line
 	6550 1250 6700 1250
@@
 Connection ~ 6550 1450
 $Comp
-L GND #PWR026
+L GND #PWR025
 U 1 1 56E9AE56
 P 6550 1600
-F 0 "#PWR026" H 6550 1600 30  0001 C CNN
+F 0 "#PWR025" H 6550 1600 30  0001 C CNN
 F 1 "GND" H 6550 1530 30  0001 C CNN
 F 2 "" H 6550 1600 60  0000 C CNN
@@
 $EndComp
 $Comp
-L +5V #PWR027
+L +5V #PWR026
 U 1 1 56E9AEAE
 P 4550 900
-F 0 "#PWR027" H 4550 990 20  0001 C CNN
+F 0 "#PWR026" H 4550 990 20  0001 C CNN
 F 1 "+5V" H 4543 1029 30  0000 C CNN
 F 2 "" H 4550 900 60  0000 C CNN
@@
 $EndComp
 $Comp
-L +3.3V #PWR028
+L +3.3V #PWR027
 U 1 1 56E9AF06
 P 5550 900
-F 0 "#PWR028" H 5550 860 30  0001 C CNN
+F 0 "#PWR027" H 5550 860 30  0001 C CNN
 F 1 "+3.3V" H 5562 1038 30  0000 C CNN
 F 2 "" H 5550 900 60  0000 C CNN
@@
 Wire Wire Line
 	9150 1150 9400 1150
+Text GLabel 8350 4700 2    60   Input ~ 0
+MOSI
+Text GLabel 9150 5050 0    60   Input ~ 0
+MOSI
+Text GLabel 8350 4900 2    60   Input ~ 0
+SLCK
+Text GLabel 9150 4900 0    60   Input ~ 0
+SLCK
+Wire Wire Line
+	8250 4700 8350 4700
+Wire Wire Line
+	8250 4900 8350 4900
+Text GLabel 8350 5100 2    60   Input ~ 0
+GPIO4
+Text GLabel 8350 5300 2    60   Input ~ 0
+GPIO5
+Wire Wire Line
+	8250 5100 8350 5100
+Wire Wire Line
+	8250 5300 8350 5300
+Text GLabel 9150 4750 0    60   Input ~ 0
+GPIO4
+Text GLabel 9150 4600 0    60   Input ~ 0
+GPIO5
+Wire Wire Line
+	9150 5200 9200 5200
+Wire Wire Line
+	9200 5200 9200 5100
+Wire Wire Line
+	9200 5100 9300 5100
+Wire Wire Line
+	9150 5050 9200 5050
+Wire Wire Line
+	9200 5050 9200 5000
+Wire Wire Line
+	9200 5000 9300 5000
+Wire Wire Line
+	9150 4900 9300 4900
+Wire Wire Line
+	9150 4750 9200 4750
+Wire Wire Line
+	9200 4750 9200 4800
+Wire Wire Line
+	9200 4800 9300 4800
+Wire Wire Line
+	9150 4600 9200 4600
+Wire Wire Line
+	9200 4600 9200 4700
+Wire Wire Line
+	9200 4700 9300 4700
 $EndSCHEMATC
